File: ppg-v1/ppg-v1.sch (KiCad schematic (older format))
At the start: 13 parts

Commit message: More schematic
Parts:
- added C? (x5): C_Small, symbol Device:C_Small
- added D?: LED_Small, symbol Device:LED_Small
- added R?: R_Small, symbol Device:R_Small
Connections:
- wire segments 17 -> 29
- no-connect marks 0 -> 2
Other:
- moved on the sheet: C?, Y?
