File: ppg-v1/ppg-v1.sch (KiCad schematic (older format))
At the start: 56 parts, among them J1 USB_microB_2040002-1, J2 Conn_01x04_Male, SW1 SW_Push, SW2 SW_Push, SW3 PCM12, U1 STM32F411CEUx, U2 MCP73831T-2ACI/OT, U3 Opamp_Dual_Generic, U4 Opamp_Dual_Generic, U5 TPS2113APW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

Commit message: Connect hardware serial pins on stm32 to Bluetooth module
Connections:
- wire segments 162 -> 154
Changed lines of the file:
@@
 EESchema Schematic File Version 4
 LIBS:ppg-v1-cache
-EELAYER 29 0
+EELAYER 26 0
 EELAYER END
 $Descr A4 11693 8268
@@
 $EndComp
 Text Label 2385 5675 2    60   ~ 0
-CTS
+RTS
 Text Label 2445 5775 2    60   ~ 0
 RST_N
 Text Label 2480 5875 2    60   ~ 0
-RTS
-Text Label 2460 5975 2    60   ~ 0
-TX
+CTS
 Text Label 3885 5275 0    60   ~ 0
-RX
+RX_IND
 Wire Wire Line
 	1930 5075 2500 5075
@@
 	2000 5275 2000 6275
 Text Label 3915 5375 0    60   ~ 0
-RX_IND
+RX
 Wire Wire Line
 	2480 5875 2500 5875
 Wire Wire Line
 	3800 5275 3885 5275
-NoConn ~ 3800 5475
 Wire Wire Line
 	1725 925  2375 925
@@
 Wire Wire Line
 	2375 925  2750 925
-Connection ~ 2500 5975
 Wire Wire Line
 	2500 5975 2510 5975
-Wire Wire Line
-	2460 5975 2500 5975
-Connection ~ 2500 5775
-Wire Wire Line
-	2500 5775 2505 5775
-Wire Wire Line
-	2445 5775 2500 5775
-Connection ~ 2500 5675
-Wire Wire Line
-	2500 5675 2505 5675
-Wire Wire Line
-	2385 5675 2500 5675
-Wire Wire Line
-	3800 5375 3915 5375
-Wire Wire Line
-	3800 5375 3795 5375
-Connection ~ 3800 5375
 NoConn ~ 3800 5975
 Wire Wire Line
@@
 Wire Wire Line
 	1810 6380 2165 6380
-Wire Wire Line
-	2165 6380 2165 5980
-Wire Wire Line
-	2165 5980 2080 5980
-Wire Wire Line
-	2080 5980 2080 6035
-Wire Wire Line
-	2080 6035 2130 6035
-Wire Wire Line
-	2130 6035 2130 5920
-Wire Wire Line
-	2130 5920 2065 5920
-Wire Wire Line
-	2065 5920 2065 5960
-Wire Wire Line
-	2065 5960 2090 5960
-Wire Wire Line
-	2090 5960 2090 5875
-Wire Wire Line
-	2090 5875 1810 5875
 Wire Wire Line
 	1810 5875 1810 5975
@@
 Wire Wire Line
 	2000 3400 2025 3400
+Wire Wire Line
+	2165 6380 2165 5875
+Wire Wire Line
+	2165 5875 1810 5875
+NoConn ~ 2510 5975
+Connection ~ 2500 5775
+Wire Wire Line
+	2500 5775 2505 5775
+Wire Wire Line
+	2445 5775 2500 5775
+Connection ~ 2500 5675
+Wire Wire Line
+	2500 5675 2505 5675
+Wire Wire Line
+	2385 5675 2500 5675
+Wire Wire Line
+	3800 5375 3915 5375
+Wire Wire Line
+	3800 5375 3795 5375
+Connection ~ 3800 5375
+Text Label 3840 5475 0    60   ~ 0
+TX
+Wire Wire Line
+	3800 5475 3840 5475
 $EndSCHEMATC
